File: kicadSchematic/rough-schematic-sketch.kicad_sch (KiCad schematic)
At the start: 25 parts, among them K1 Compressor Relay, K2 Auger Relay, M1 Compressor, M2 Auger Motor, M3 Pump, M4 Fan, Q1 Pump Mosfet, Q2 UV LED Mosfet, Q3 Fan Mosfet, SW1 Reset Button, SW2 Power Switch, SW3 Bin Switch, SW4 Float High, SW5 Float Low

Commit message: hooked up IR LED, reverse engineering details of front panel
Parts:
- R4: value 10kΩ -> 1MΩ
Connections:
- net at R3.1, R4.1: now also A1.20 (A1); no longer A1.16 (D13)
Other:
- note added: "When active, will hit about 1.6v"
Changed lines of the file:
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@@
+		)
+	)
+	(text "When active, will hit about 1.6v"
+		(exclude_from_sim no)
+		(at 149.606 149.098 0)
+		(effects
+			(font
+				(size 1.27 1.27)
+			)
 		)
 	)
@@
 	(wire
 		(pts
-			(xy 149.86 160.02) (xy 144.78 160.02)
-		)
-		(stroke
-			(width 0)
-			(type default)
-		)
-	)
-	(wire
-		(pts
 			(xy 110.49 99.06) (xy 110.49 135.89)
 		)
@@
 	(wire
 		(pts
-			(xy 149.86 146.05) (xy 149.86 160.02)
-		)
-		(stroke
-			(width 0)
-			(type default)
-		)
-	)
-	(wire
-		(pts
 			(xy 104.14 88.9) (xy 104.14 91.44)
 		)
@@
 	(wire
 		(pts
+			(xy 144.78 160.02) (xy 170.18 160.02)
+		)
+		(stroke
+			(width 0)
+			(type default)
+		)
+	)
+	(wire
+		(pts
 			(xy 91.44 82.55) (xy 90.17 82.55)
 		)
@@
 	(wire
 		(pts
-			(xy 132.08 111.76) (xy 132.08 146.05)
+			(xy 170.18 96.52) (xy 157.48 96.52)
 		)
 		(stroke
@@
 	(wire
 		(pts
+			(xy 170.18 160.02) (xy 170.18 96.52)
+		)
+		(stroke
+			(width 0)
+			(type default)
+		)
+	)
+	(wire
+		(pts
 			(xy 186.69 134.62) (xy 124.46 134.62)
-		)
-		(stroke
-			(width 0)
-			(type default)
-		)
-	)
-	(wire
-		(pts
-			(xy 132.08 146.05) (xy 149.86 146.05)
 		)
 		(stroke
@@
 			)
 		)
-		(property "Value" "10kΩ"
+		(property "Value" "1MΩ"
 			(at 147.32 165.0999 0)
 			(show_name no)

Commit message: I think I've been committing to the internal firmware git repo
Parts:
- removed SW1: Reset Button, symbol Switch:SW_Push
- removed SW2: Power Switch, symbol Switch:SW_SPST
- added J1: Front Panel, symbol Connector_Generic:Conn_01x04
Connections:
- net +5V: now also J1.4 (Pin_4)
- net GND: now also J1.3 (Pin_3)
- net SDA: now reaches A1.23 (A4)
- net SDA: now also J1.1 (Pin_1)
- net SCK: now reaches A1.24 (A5)
- net SCK: now also J1.2 (Pin_2)
